Commit message: Added point cloud sensor

File: turtlebot3_gazebo/urdf/turtlebot3_burger_cam.urdf (robot description, URDF)
Before this commit: robot turtlebot3_burger_cam, 10 links, 9 joints
Links:
- added link burger_cam/camera_link/depth_camera
Joints:
- added joint camera_depth_joint: type fixed, parent camera_link, child burger_cam/camera_link/depth_camera, origin xyz=0 0 0 rpy=0 0 0
