Commit message: fix: Missing prefix in joint name

File: projects/turtlebot3_descriptions/urdf/turtlebot3_burger_oak_d_pro.urdf (robot description, URDF)
Before this commit: robot turtlebot3_burger, 10 links, 9 joints
Joints:
- removed joint oak_d_pro_depth_optical_frame
- added joint joint_oak_d_pro_depth_optical_frame: type fixed, parent oak_d_pro_camera, child oak_d_pro_depth_optical_frame, origin xyz=0.0 0.0 0.0 rpy=-1.5708 0.0 -1.5708
